Commit message: refactor: change angular speed, launch file, robot color

File: my_robot/urdf/my_robot.xacro (robot description, xacro)
@@ -10,5 +10,5 @@
   <link name='chassis'>
     <pose>0 0 0.1 0 0 0</pose>
-    <inertial>
+    <inertial name="chassis_visual">
       <mass value="15.0"/>
       <origin xyz="0.0 0 0" rpy=" 0 0 0"/>
@@ -16,8 +16,7 @@
           ixx="0.1" ixy="0" ixz="0"
           iyy="0.1" iyz="0"
-          izz="0.1"
-      />
+          izz="0.1"/>
     </inertial>
-    <collision name='collision'>
+    <collision name='chassis_collision'>
       <origin xyz="0 0 0" rpy=" 0 0 0"/>
       <geometry>
@@ -60,10 +59,32 @@
   </link>
   <link name="left_wheel">
-  <inertial>
+  <inertial name="left_wheel_inertial">
   <mass value="5.0"/>
   <origin xyz="0 0 0" rpy="0.0 1.5707 1.5707"/>
   <inertia ixx="0.1" ixy="0" ixz="0" iyy="0.1" iyz="0" izz="0.1"/>
   </inertial>
-  <collision>
+  <collision name="left_wheel_collision">
+  <origin xyz="0 0 0" rpy="0.0 1.5707 1.5707"/>
+  <geometry>
+  <cylinder  radius="0.1" length="0.05" />
+  </geometry>
+  </collision>
+  <visual name="left_wheel_visual">
+  <origin xyz="0 0 0" rpy="0.0 1.5707 1.5707"/>
+  <geometry>
+  <cylinder  radius="0.1" length="0.05" />
+  </geometry>
+  <material name="Green">
+    <color rgba="0 1 0 1" />
+  </material>
+  </visual>
+  </link>
+  <link name="right_wheel">
+  <inertial name="right_wheel_inertial">
+  <mass value="5.0"/>
+  <origin xyz="0 0 0" rpy="0.0 1.5707 1.5707"/>
+  <inertia ixx="0.1" ixy="0" ixz="0" iyy="0.1" iyz="0" izz="0.1"/>
+  </inertial>
+  <collision name="right_wheel_collision">
   <origin xyz="0 0 0" rpy="0.0 1.5707 1.5707"/>
   <geometry>
@@ -76,28 +97,6 @@
   <cylinder  radius="0.1" length="0.05" />
   </geometry>
-  <material name="Black">
-    <color rgba="0 0 0 1" />
-  </material>
-  </visual>
-  </link>
-  <link name="right_wheel">
-  <inertial>
-  <mass value="5.0"/>
-  <origin xyz="0 0 0" rpy="0.0 1.5707 1.5707"/>
-  <inertia ixx="0.1" ixy="0" ixz="0" iyy="0.1" iyz="0" izz="0.1"/>
-  </inertial>
-  <collision>
-  <origin xyz="0 0 0" rpy="0.0 1.5707 1.5707"/>
-  <geometry>
-  <cylinder  radius="0.1" length="0.05" />
-  </geometry>
-  </collision>
-  <visual>
-  <origin xyz="0 0 0" rpy="0.0 1.5707 1.5707"/>
-  <geometry>
-  <cylinder  radius="0.1" length="0.05" />
-  </geometry>
-  <material name="Black">
-    <color rgba="0 0 0 1" />
+  <material name="Green">
+    <color rgba="0 1 0 1" />
   </material>
   </visual>
@@ -109,5 +108,5 @@
 <inertia ixx="1e-6" ixy="0" ixz="0" iyy="1e-6" iyz="0" izz="1e-6" />
 </inertial>
-<collision>
+<collision name="camera_collision">
 <origin xyz="0 0 0" rpy="0 0 0"/>
 <geometry>
@@ -115,5 +114,5 @@
 </geometry>
 </collision>
-<visual>
+<visual name="camera_visual">
 <origin xyz="0 0 0" rpy="0 0 0"/>
 <geometry>

Commit message: refactor: update robot model and show color

File: my_robot/urdf/my_robot.xacro (robot description, xacro)
@@ -21,5 +21,5 @@
       <origin xyz="0 0 0" rpy=" 0 0 0"/>
       <geometry>
-        <box size=".4 .2 .1"/>
+        <box size=".2 .2 .1"/>
       </geometry>
     </collision>
@@ -27,5 +27,5 @@
       <origin xyz="0 0 0" rpy=" 0 0 0"/>
       <geometry>
-        <box size=".4 .2 .1"/>
+        <box size=".2 .2 .1"/>
       </geometry>
     <material name="blue">
@@ -33,18 +33,6 @@
     </material>
     </visual>
-    <collision name='back_caster_collision'>
-      <origin xyz="-0.15 0 -0.05" rpy=" 0 0 0"/>
-      <geometry>
-        <sphere radius="0.0499"/>
-      </geometry>
-    </collision>
-    <visual name='back_caster_visual'>
-      <origin xyz="-0.15 0 -0.05" rpy=" 0 0 0"/>
-      <geometry>
-        <sphere radius="0.05"/>
-      </geometry>
-    </visual>
     <collision name='front_caster_collision'>
-      <origin xyz="0.15 0 -0.05" rpy=" 0 0 0"/>
+      <origin xyz="0.05 0 -0.05" rpy=" 0 0 0"/>
       <geometry>
         <sphere radius="0.0499"/>
@@ -52,5 +40,5 @@
     </collision>
     <visual name='front_caster_visual'>
-      <origin xyz="0.15 0 -0.05" rpy=" 0 0 0"/>
+      <origin xyz="0.05 0 -0.05" rpy=" 0 0 0"/>
       <geometry>
         <sphere radius="0.05"/>
@@ -67,5 +55,5 @@
   <origin xyz="0 0 0" rpy="0.0 1.5707 1.5707"/>
   <geometry>
-  <cylinder  radius="0.1" length="0.05" />
+  <cylinder  radius="0.05" length="0.01" />
   </geometry>
   </collision>
@@ -73,5 +61,5 @@
   <origin xyz="0 0 0" rpy="0.0 1.5707 1.5707"/>
   <geometry>
-  <cylinder  radius="0.1" length="0.05" />
+  <cylinder  radius="0.05" length="0.01" />
   </geometry>
   <material name="Green">
@@ -89,5 +77,5 @@
   <origin xyz="0 0 0" rpy="0.0 1.5707 1.5707"/>
   <geometry>
-  <cylinder  radius="0.1" length="0.05" />
+  <cylinder  radius="0.05" length="0.01" />
   </geometry>
   </collision>
@@ -95,5 +83,5 @@
   <origin xyz="0 0 0" rpy="0.0 1.5707 1.5707"/>
   <geometry>
-  <cylinder  radius="0.1" length="0.05" />
+  <cylinder  radius="0.05" length="0.01" />
   </geometry>
   <material name="Green">
@@ -144,5 +132,5 @@
 </link>
 <joint type="fixed" name="hokuyo_joint">
-<origin xyz="0.15 0 0.1" rpy="0 0 0"/>
+<origin xyz="0.05 0 0.1" rpy="0 0 0"/>
 <parent link="chassis"/>
 <child link="hokuyo"/>
@@ -150,5 +138,5 @@
 </joint>
 <joint type="fixed" name="camera_joint">
-<origin xyz="0.2 0 0" rpy="0 0 0" />
+<origin xyz="0.1 0 0" rpy="0 0 0" />
 <parent link="chassis"/>
 <child link="camera" />
@@ -156,5 +144,5 @@
 </joint>
 <joint type="continuous" name="right_wheel_hinge">
-<origin xyz="0 -0.15 0" rpy="0 0 0" />
+<origin xyz="-0.1 -0.11 -0.05" rpy="0 0 0" />
 <child link="right_wheel" />
 <parent link="chassis" />
@@ -164,5 +152,5 @@
 </joint>
 <joint type="continuous" name="left_wheel_hinge">
-<origin xyz="0 0.15 0" rpy="0 0 0" />
+<origin xyz="-0.1 0.11 -0.05" rpy="0 0 0" />
 <child link="left_wheel" />
 <parent link="chassis" />
@@ -171,3 +159,42 @@
 <dynamics damping="1.0" friction="1.0" />
 </joint>
+<material name="Blue">
+    <color rgba="0.0 0.0 0.8 1.0"/>
+  </material>
+  <material name="Green">
+    <color rgba="0.0 0.8 0.0 1.0"/>
+  </material>
+  <material name="Grey">
+    <color rgba="0.7 0.7 0.7 1.0"/>
+  </material>
+  <material name="Grey2">
+    <color rgba="0.9 0.9 0.9 1.0"/>
+  </material>
+  <material name="Red">
+    <color rgba="0.8 0.0 0.0 1.0"/>
+  </material>
+  <material name="White">
+    <color rgba="1.0 1.0 1.0 1.0"/>
+  </material>
+  <material name="Black">
+    <color rgba="0.1 0.1 0.1 1.0"/>
+  </material>
+  <material name="LightGrey">
+    <color rgba="0.6 0.6 0.6 1.0"/>
+  </material>
+  <material name="Orange">
+    <color rgba="1.0 0.33 0.0 1.0"/>
+  </material>
+<gazebo reference="left_wheel">
+<material>Gazebo/Green</material>
+</gazebo>
+<gazebo reference="right_wheel">
+<material>Gazebo/Green</material>
+</gazebo>
+<gazebo reference="camera">
+<material>Gazebo/Blue</material>
+</gazebo>
+<gazebo reference="chassis">
+<material>Gazebo/Orange</material>
+</gazebo>
 </robot>
